Commit message: [rapiro_description] Complete URDF model of Rapiro including STL meshes.

File: rapiro_description/urdf/rapiro.urdf (robot description, URDF)
Before this commit: robot rapiro, 9 links, 8 joints
Links:
- added link l_arm; visual mesh filename=package://rapiro_description/meshes/l_arm.stl
- added link l_hand; visual mesh filename=package://rapiro_description/meshes/l_hand.stl
- added link l_shoulder; visual mesh filename=package://rapiro_description/meshes/shoulder.stl
- added link r_arm; visual mesh filename=package://rapiro_description/meshes/r_arm.stl
- added link r_hand; visual mesh filename=package://rapiro_description/meshes/r_hand.stl
- added link r_shoulder; visual mesh filename=package://rapiro_description/meshes/shoulder.stl
- link body: geometry visual mesh filename=package://rapiro_description/meshes/backpack.stl; visual mesh filename=package://rapiro_description/meshes/body.stl
Joints:
- added joint l_hand_jnt: type revolute, parent l_arm, child l_hand, origin xyz=.0505 0 0 rpy=3.142 0 .960, axis 0 0 1, limit lower=0 upper=3.142 effort=1000.0 velocity=10
- added joint l_shld_p_jnt: type revolute, parent l_shoulder, child l_arm, origin xyz=0 0 .0225 rpy=1.571 .873 0, axis 0 0 1, limit lower=0 upper=3.142 effort=1000.0 velocity=10
- added joint l_shld_r_jnt: type revolute, parent body, child l_shoulder, origin xyz=0 .06 .0225 rpy=0 -1.571 -1.571, axis 0 0 1, limit lower=0 upper=3.142 effort=1000.0 velocity=10
- added joint r_hand_jnt: type revolute, parent r_arm, child r_hand, origin xyz=.0505 0 0 rpy=3.142 0 1.920, axis 0 0 1, limit lower=0 upper=3.142 effort=1000.0 velocity=10
- added joint r_shld_p_jnt: type revolute, parent r_shoulder, child r_arm, origin xyz=0 0 .0225 rpy=-1.571 -2.269 0, axis 0 0 1, limit lower=0 upper=3.142 effort=1000.0 velocity=10
- added joint r_shld_r_jnt: type revolute, parent body, child r_shoulder, origin xyz=0 -.06 .0225 rpy=0 1.571 -1.571, axis 0 0 1, limit lower=0 upper=3.142 effort=1000.0 velocity=10

Commit message: [rapiro_arduino][rapiro_description] Adjust joint limits.

File: rapiro_description/urdf/rapiro.urdf (robot description, URDF)
Before this commit: robot rapiro, 15 links, 14 joints
Joints:
- joint l_hand_jnt: limit lower=0 upper=3.142 effort=1000.0 velocity=10 -> lower=.960 upper=1.920 effort=1000.0 velocity=10
- joint l_shld_p_jnt: limit lower=0 upper=3.142 effort=1000.0 velocity=10 -> lower=.785 upper=2.705 effort=1000.0 velocity=10
- joint r_hand_jnt: limit lower=0 upper=3.142 effort=1000.0 velocity=10 -> lower=.960 upper=1.920 effort=1000.0 velocity=10
- joint r_shld_p_jnt: limit lower=0 upper=3.142 effort=1000.0 velocity=10 -> lower=.436 upper=2.356 effort=1000.0 velocity=10

Commit message: [rapiro_description] Attach base_link to body instead of waist.

File: rapiro_description/urdf/rapiro.urdf (robot description, URDF)
Before this commit: robot rapiro, 15 links, 14 joints
Joints:
- removed joint base_waist_fix
- added joint base_fix: type fixed, parent base_link, child body
- joint l_foot_y_jnt: origin xyz=0 .03 -.015 rpy=3.142 0 1.571 -> xyz=0 -.03 .015 rpy=0 0 -1.571
- joint r_foot_y_jnt: origin xyz=0 -.03 -.015 rpy=3.142 0 1.571 -> xyz=0 .03 .015 rpy=0 0 -1.571
- joint waist_jnt: child body -> waist; origin xyz=0 0 .015 rpy=0 0 -1.571 -> xyz=0 0 -.015 rpy=3.142 0 1.571; parent waist -> body

Commit message: [rapiro_cmd] Add Odometry for Rapiro. Values are estimated based on movement of feet.

File: rapiro_description/urdf/rapiro.urdf (robot description, URDF)
Before this commit: robot rapiro, 15 links, 14 joints
Joints:
- joint base_waist_fix: origin (none) -> xyz=0 0 .065
